Commit message: feat: Add spawn_preset parameter and align sensor topics with real robot
- Add spawn_preset arg to limo_ackerman.launch (default, m2)
- Adjust camera position (2cm forward, 3cm up, 20deg down)
- Change IMU topic from /limo/imu to /imu
- Adjust LiDAR samples from 720 to 378
- Remove imu_orientation_adapter node

File: limo_description/urdf/limo_ackerman.xacro (robot description, xacro)
@@ -56,5 +56,5 @@
     </xacro:limo_laser>
     <xacro:limo_depth_camera parent_prefix="base_link" frame_prefix="depth_camera">
-        <origin xyz="0.084 0 0.03" rpy="0 0 0"/>
+        <origin xyz="0.114 0 0.06" rpy="0 0.35 0"/>
     </xacro:limo_depth_camera>
     <xacro:limo_imu parent_prefix="base_link" frame_prefix="imu">
